File: MCU Datalogger.kicad_sch (KiCad schematic)
At the start: 0 parts

Commit message: Have required added symbols on the sheets
Parts:
- added BT1: Battery, symbol Device:Battery
- added C1, C2, C3, C4: C, symbol Device:C
- added C5: C_Polarized, symbol Device:C_Polarized
- added D1, D2: LED, symbol Device:LED
- added H1, H2, H3, H4: MountingHole, symbol Mechanical:MountingHole
- added R1, R2, R3, R4, R5, R6, R7: R, symbol Device:R
- added U1, U2: 24LC1025, symbol Memory_EEPROM:24LC1025
- added U3, U4: DS1337S_, DS1337S_:SOIC127P600X175-8N, symbol DS1337S_:DS1337S_
- added U5: ATMEGA328P-AUR, ATMEGA328P-AUR:QFP80P900X900X120-32N, symbol ATMEGA328P-AUR:ATMEGA328P-AUR
- added Y1, Y2: Crystal, symbol Device:Crystal
Connections:
- new net GND: U5.21 (GND), U5.3 (GND), U5.5 (GND)
- new net VCC: U5.4 (VCC), U5.6 (VCC)
Other:
- added sheet Connecters (connectors.kicad_sch)
